Commit message: urdf 수정

File: src/nav2_wheel/urdf/model.xacro (robot description, xacro)
@@ -37,5 +37,5 @@
             <origin xyz="0 0 0"/>
             <geometry>
-                <cylinder radius="0.3" length="0.11"/>
+                <cylinder radius="0.1" length="0.11"/>
             </geometry>
             <material name="blue"/>
@@ -44,8 +44,8 @@
             <origin xyz="0 0 0"/>
             <geometry>
-                <cylinder radius="0.3" length="0.11"/>
+                <cylinder radius="0.1" length="0.11"/>
             </geometry>
         </collision>
-        <xacro:inertial_cylinder mass="0.5" length="0.11" radius="0.3">
+        <xacro:inertial_cylinder mass="0.5" length="0.11" radius="0.1">
             <origin xyz="0 0 0" rpy="0 0 0"/>
         </xacro:inertial_cylinder>
@@ -54,5 +54,5 @@
         <parent link="base_link"/>
         <child link="wheel_left"/>
-        <origin xyz="-0.2 0.28 0.0395" rpy="1.57 0 0" />
+        <origin xyz="0.2 0.28 0" rpy="1.57 0 0" />
         <axis xyz="0 0 1"/>
     </joint>
@@ -61,5 +61,5 @@
             <origin xyz="0 0 0"/>
             <geometry>
-                <cylinder radius="0.3" length="0.11"/>
+                <cylinder radius="0.1" length="0.11"/>
             </geometry>
             <material name="blue"/>
@@ -68,8 +68,8 @@
             <origin xyz="0 0 0"/>
             <geometry>
-                <cylinder radius="0.3" length="0.11"/>
+                <cylinder radius="0.1" length="0.11"/>
             </geometry>
         </collision>
-        <xacro:inertial_cylinder mass="0.5" length="0.11" radius="0.3">
+        <xacro:inertial_cylinder mass="0.5" length="0.11" radius="0.1">
             <origin xyz="0 0 0" rpy="0 0 0"/>
         </xacro:inertial_cylinder>
@@ -78,5 +78,5 @@
         <parent link="base_link"/>
         <child link="wheel_right"/>
-        <origin xyz="-0.2 -0.28 0.0395" rpy="1.57 0 0" />
+        <origin xyz="0.2 -0.28 0" rpy="1.57 0 0" />
         <axis xyz="0 0 1"/>
     </joint>
@@ -101,5 +101,5 @@
         <parent link="base_link"/>
         <child link="caster_wheel"/>
-        <origin xyz="0.2 0 0"/>
+        <origin xyz="-0.2 0 0"/>
     </joint>
     <link name="laser_frame"/>
